Commit message: Feat: incorporate rein's nav2 into current ws, fix imu_fixer according to rein's

File: src/amr_description/urdf/amr.urdf.xacro (robot description, xacro)
@@ -175,4 +175,17 @@
     </plugin>
   </gazebo>
+  <!-- ============ VIRTUAL MERGED LASER FRAME ============ -->
+  <link name="laser_frame">
+    <inertial>
+      <mass value="0.001"/>
+      <inertia ixx="1e-6" ixy="0" ixz="0" iyy="1e-6" iyz="0" izz="1e-6"/>
+    </inertial>
+  </link>
+  <joint name="laser_frame_joint" type="fixed">
+    <parent link="base_link"/>
+    <child  link="laser_frame"/>
+    <!-- Position the virtual merged frame at top plate center (Z = lidar_z_off) -->
+    <origin xyz="0.0 0.0 ${lidar_z_off}" rpy="0 0 0"/>
+  </joint>
   <!-- ============ LIDAR ============ -->
   <!-- Mesh lidar punya bottom di Z=0 setelah rotasi. Visual origin Z=-0.032 agar
