Commit message: refactor: update launch files, add ROS-Gazebo bridge configuration, and implement simple scan merger

File: src/description/amr_description/urdf/amr.urdf.xacro (robot description, xacro)
@@ -61,5 +61,11 @@
     <origin xyz="0 0 ${wheel_radius}" rpy="0 0 0"/>
   </joint>
-  <link name="base_link">
+  <link name="base_link"/>
+  <joint name="base_link_joint" type="fixed">
+    <parent link="base_link"/>
+    <child  link="chassis_link"/>
+    <origin xyz="-0.05 0 0" rpy="0 0 0"/>
+  </joint>
+  <link name="chassis_link">
     <!-- Mesh di-shift ke atas agar bottom-nya pas di Z=0 base_link -->
     <visual>
@@ -156,21 +162,24 @@
   </gazebo>
   <gazebo>
-    <plugin name="diff_drive" filename="libgazebo_ros_diff_drive.so">
-      <ros>
-        <remapping>cmd_vel:=cmd_vel</remapping>
-        <remapping>odom:=odom</remapping>
-      </ros>
+    <plugin filename="gz-sim-diff-drive-system" name="gz::sim::systems::DiffDrive">
       <left_joint>wheel_left_joint</left_joint>
       <right_joint>wheel_right_joint</right_joint>
       <wheel_separation>${wheel_separation}</wheel_separation>
-      <wheel_diameter>${2*wheel_radius}</wheel_diameter>
-      <max_wheel_torque>50000.0</max_wheel_torque>
-      <max_wheel_acceleration>10.0</max_wheel_acceleration>
-      <publish_odom>true</publish_odom>
-      <publish_odom_tf>true</publish_odom_tf>
-      <publish_wheel_tf>true</publish_wheel_tf>
-      <publish_wheel_joint_state>true</publish_wheel_joint_state>
-      <odometry_frame>odom</odometry_frame>
-      <robot_base_frame>base_footprint</robot_base_frame>
+      <wheel_radius>${wheel_radius}</wheel_radius>
+      <max_linear_acceleration>10.0</max_linear_acceleration>
+      <max_angular_acceleration>10.0</max_angular_acceleration>
+      <topic>cmd_vel</topic>
+      <odom_topic>odom</odom_topic>
+      <tf_topic>tf</tf_topic>
+      <frame_id>odom</frame_id>
+      <child_frame_id>base_footprint</child_frame_id>
+      <odom_publisher_frequency>30</odom_publisher_frequency>
+    </plugin>
+    <plugin filename="gz-sim-joint-state-publisher-system" name="gz::sim::systems::JointStatePublisher">
+      <topic>joint_states</topic>
+      <joint_name>wheel_left_joint</joint_name>
+      <joint_name>wheel_right_joint</joint_name>
+    </plugin>
+    <plugin filename="gz-sim-sensors-system" name="gz::sim::systems::Sensors">
     </plugin>
   </gazebo>
@@ -200,9 +209,11 @@
     <gazebo reference="${name}_link">
       <material>Gazebo/Blue</material>
-      <sensor name="${name}_sensor" type="ray">
+      <sensor name="${name}_sensor" type="gpu_lidar">
         <always_on>true</always_on>
         <visualize>true</visualize>
         <update_rate>10</update_rate>
-        <ray>
+        <topic>${topic_name}</topic>
+        <gz_frame_id>${name}_link</gz_frame_id>
+        <lidar>
           <scan>
             <horizontal>
@@ -212,10 +223,5 @@
           </scan>
           <range><min>0.15</min><max>12.0</max><resolution>0.01</resolution></range>
-        </ray>
-        <plugin name="${name}_plugin" filename="libgazebo_ros_ray_sensor.so">
-          <ros><remapping>~/out:=${topic_name}</remapping></ros>
-          <output_type>sensor_msgs/LaserScan</output_type>
-          <frame_name>${name}_link</frame_name>
-        </plugin>
+        </lidar>
       </sensor>
     </gazebo>
@@ -247,9 +253,9 @@
       <material>Gazebo/Green</material>
       <sensor name="${name}_sensor" type="imu">
-        <always_on>true</always_on><update_rate>50</update_rate>
-        <plugin name="${name}_plugin" filename="libgazebo_ros_imu_sensor.so">
-          <ros><remapping>~/out:=/imu/data</remapping></ros>
-          <initial_orientation_as_reference>false</initial_orientation_as_reference>
-        </plugin>
+        <always_on>true</always_on>
+        <update_rate>50</update_rate>
+        <topic>imu/data</topic>
+        <gz_frame_id>${name}_link</gz_frame_id>
+        <imu/>
       </sensor>
     </gazebo>

Commit message: feat: add simulation package with Gazebo integration and ROS-Gazebo bridge configuration fix: fix robot description

File: src/description/amr_description/urdf/amr.urdf.xacro (robot description, xacro)
@@ -4,29 +4,29 @@
        base_link mesh: ukuran 1.0x1.0x0.519, bottom di Z=-0.118 (sebelum kompensasi). -->
   <!-- ============ PROPERTIES ============ -->
-  <xacro:property name="body_length" value="1.00"/>
-  <xacro:property name="body_width"  value="1.00"/>
-  <xacro:property name="body_height" value="0.519"/>
+  <xacro:property name="body_length" value="0.66"/>
+  <xacro:property name="body_width"  value="0.62"/>
+  <xacro:property name="body_height" value="0.200"/>
   <xacro:property name="body_mass"   value="80.0"/>
   <!-- Shift visual base mesh ke atas: bottom mesh asli ada di Z=-0.118 setelah rotasi -->
   <xacro:property name="base_mesh_z_shift" value="0.118"/>
-  <xacro:property name="wheel_radius"     value="0.105"/>
-  <xacro:property name="wheel_width"      value="0.04"/>
+  <xacro:property name="wheel_radius"     value="0.065"/>
+  <xacro:property name="wheel_width"      value="0.055"/>
   <xacro:property name="wheel_mass"       value="3.0"/>
-  <xacro:property name="wheel_separation" value="0.58"/>
-  <xacro:property name="caster_radius" value="0.05"/>
+  <xacro:property name="wheel_separation" value="0.45"/>
+  <xacro:property name="caster_radius" value="0.065"/>
   <xacro:property name="caster_mass"   value="0.45"/>
-  <xacro:property name="caster_x_front" value=" 0.29"/>
+  <xacro:property name="caster_x_front" value=" 0.21"/>
   <xacro:property name="caster_x_rear"  value="-0.29"/>
-  <xacro:property name="caster_y_outer" value=" 0.29"/>
+  <xacro:property name="caster_y_outer" value=" 0.225"/>
   <!-- Lidar di pojok diagonal body, sedikit di atas top plate -->
   <xacro:property name="lidar_x_off" value="0.45"/>
   <xacro:property name="lidar_y_off" value="0.45"/>
-  <xacro:property name="lidar_z_off" value="0.25"/>
-  <xacro:property name="lidar_x"    value="0.064"/>
-  <xacro:property name="lidar_y"    value="0.064"/>
-  <xacro:property name="lidar_z"    value="0.065"/>
+  <xacro:property name="lidar_z_off" value="0.2"/>
+  <xacro:property name="lidar_x"    value="0.035"/>
+  <xacro:property name="lidar_y"    value="0.035"/>
+  <xacro:property name="lidar_z"    value="0.01"/>
   <xacro:property name="lidar_mass" value="0.10"/>
   <xacro:property name="mesh_pkg" value="package://amr_description/meshes"/>
-  <xacro:property name="mesh_rpy_base" value="1.5708 0 -1.5708"/>
+  <xacro:property name="mesh_rpy_base" value="1.5708 0 1.5708"/>
   <!-- ============ INERTIA MACROS ============ -->
   <xacro:macro name="box_inertia" params="m x y z">
@@ -86,5 +86,5 @@
     <link name="wheel_${name}_link">
       <visual>
-        <origin xyz="0 ${y_shift} -0.014" rpy="${mesh_rpy_base}"/>
+        <origin xyz="0 ${y_shift} 0" rpy="${mesh_rpy_base}"/>
         <geometry><mesh filename="${mesh_pkg}/${mesh_file}"/></geometry>
         <material name="wheel_black"><color rgba="0.15 0.15 0.15 1.0"/></material>
@@ -112,5 +112,5 @@
     <link name="caster_${name}_link">
       <visual>
-        <origin xyz="0 0 -0.014" rpy="${mesh_rpy_base}"/>
+        <origin xyz="0 0 0" rpy="${mesh_rpy_base}"/>
         <geometry><mesh filename="${mesh_pkg}/${mesh_file}"/></geometry>
         <material name="caster_silver"><color rgba="0.75 0.75 0.75 1.0"/></material>
@@ -122,5 +122,5 @@
       <parent link="base_link"/>
       <child  link="caster_${name}_link"/>
-      <origin xyz="${xp} ${yp} ${-wheel_radius+caster_radius}" rpy="0 0 0"/>
+      <origin xyz="${xp} ${yp} 0" rpy="0 0 0"/>
     </joint>
     <gazebo reference="caster_${name}_link">
@@ -190,10 +190,10 @@
     <link name="${name}_link">
       <visual>
-        <origin xyz="0 0 -0.032" rpy="${mesh_rpy_base}"/>
-        <geometry><mesh filename="${mesh_pkg}/${mesh_file}"/></geometry>
+        <origin xyz="0 0 -0.03" rpy="1.5708 0 ${yaw+3.14159}"/>
+        <!-- <geometry><mesh filename="${mesh_pkg}/${mesh_file}"/></geometry> -->
         <material name="lidar_blue"><color rgba="0.0 0.2 0.8 1.0"/></material>
       </visual>
       <collision>
-        <geometry><box size="${lidar_x} ${lidar_y} ${lidar_z}"/></geometry>
+        <geometry><cylinder radius="0.0175" length="${lidar_z}"/></geometry>
       </collision>
       <inertial>
@@ -228,9 +228,9 @@
   </xacro:macro>
   <xacro:lidar_sensor name="lidar_front_right"
-                      xp=" 0.31" yp="-0.32" yaw="${-pi/4}"
-                      topic_name="scan_front" mesh_file="lidar1_link.stl"/>
+                      xp="0.32" yp="-0.31" yaw="${-pi/4}"
+                      topic_name="front_scan" mesh_file="lidar1_link.stl"/>
   <xacro:lidar_sensor name="lidar_rear_left"
-                      xp="-0.31" yp=" 0.42" yaw="${3*pi/4}"
-                      topic_name="scan_rear" mesh_file="lidar2_link.stl"/>
+                      xp="-0.42" yp="0.31" yaw="${3*pi/4}"
+                      topic_name="rear_scan" mesh_file="lidar2_link.stl"/>
   <!-- ============ IMU ============ -->
   <xacro:macro name="imu_sensor" params="name xp yp">

Commit message: refactor: update URDF properties for body dimensions and caster offsets; add RViz configuration file

File: src/description/amr_description/urdf/amr.urdf.xacro (robot description, xacro)
@@ -4,7 +4,7 @@
        base_link mesh: ukuran 1.0x1.0x0.519, bottom di Z=-0.118 (sebelum kompensasi). -->
   <!-- ============ PROPERTIES ============ -->
-  <xacro:property name="body_length" value="0.66"/>
-  <xacro:property name="body_width"  value="0.62"/>
-  <xacro:property name="body_height" value="0.200"/>
+  <xacro:property name="body_length" value="1.0"/>
+  <xacro:property name="body_width"  value="1.0"/>
+  <xacro:property name="body_height" value="0.27"/>
   <xacro:property name="body_mass"   value="80.0"/>
   <!-- Shift visual base mesh ke atas: bottom mesh asli ada di Z=-0.118 setelah rotasi -->
@@ -16,7 +16,7 @@
   <xacro:property name="caster_radius" value="0.065"/>
   <xacro:property name="caster_mass"   value="0.45"/>
-  <xacro:property name="caster_x_front" value=" 0.21"/>
-  <xacro:property name="caster_x_rear"  value="-0.29"/>
-  <xacro:property name="caster_y_outer" value=" 0.225"/>
+  <xacro:property name="caster_x_front" value=" 0.23"/>
+  <xacro:property name="caster_x_rear"  value="-0.4"/>
+  <xacro:property name="caster_y_outer" value=" 0.29"/>
   <!-- Lidar di pojok diagonal body, sedikit di atas top plate -->
   <xacro:property name="lidar_x_off" value="0.45"/>
@@ -191,5 +191,5 @@
       <visual>
         <origin xyz="0 0 -0.03" rpy="1.5708 0 ${yaw+3.14159}"/>
-        <!-- <geometry><mesh filename="${mesh_pkg}/${mesh_file}"/></geometry> -->
+        <geometry><mesh filename="${mesh_pkg}/${mesh_file}"/></geometry>
         <material name="lidar_blue"><color rgba="0.0 0.2 0.8 1.0"/></material>
       </visual>
